File: hardware/LEDHeart/power.kicad_sch (KiCad schematic)
At the start: 24 parts, among them Q1 MMBT3904, Q2 AO3401A, Q3 MMBT3904, U2 TPS61222DCK, U3 CH32V003JxMx

Commit message: Couple More effects
Parts:
- C9: value 10uF -> 2.2uF
- R10: value 10K -> 200K
Changed lines of the file:
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@@
 			)
 		)
-		(property "Value" "10uF"
+		(property "Value" "2.2uF"
 			(at 137.16 55.8799 0)
 			(show_name no)
@@
 			)
 		)
-		(property "Value" "10K"
+		(property "Value" "200K"
 			(at 144.78 66.0399 0)
 			(show_name no)

Commit message: Some hardware updates
Parts:
- added R15: 1M, Resistor_SMD:R_0402_1005Metric, symbol Device:R
Connections:
- net at C9.1, Q3.1 (B), R11.2: now also R15.1
- net at C9.2, Q3.2 (E), R10.1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: now also R15.2
Other:
- moved on the sheet: R11
Changed lines of the file:
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@@
+	)
+	(junction
+		(at 123.19 48.26)
+		(diameter 0)
+		(color 0 0 0 0)
 	)
 	(junction
@@
 	)
 	(junction
+		(at 133.35 58.42)
+		(diameter 0)
+		(color 0 0 0 0)
+	)
+	(junction
 		(at 27.94 54.61)
+		(diameter 0)
+		(color 0 0 0 0)
+	)
+	(junction
+		(at 133.35 48.26)
 		(diameter 0)
 		(color 0 0 0 0)
@@
 	)
 	(junction
-		(at 133.35 48.26)
-		(diameter 0)
-		(color 0 0 0 0)
-	)
-	(junction
 		(at 58.42 97.79)
 		(diameter 0)
@@
 	(wire
 		(pts
-			(xy 107.95 48.26) (xy 123.19 48.26)
+			(xy 107.95 48.26) (xy 115.57 48.26)
 		)
 		(stroke
@@
 	(wire
 		(pts
+			(xy 123.19 58.42) (xy 123.19 57.15)
+		)
+		(stroke
+			(width 0)
+			(type default)
+		)
+	)
+	(wire
+		(pts
 			(xy 142.24 30.48) (xy 153.67 30.48)
 		)
@@
 	(wire
 		(pts
-			(xy 130.81 48.26) (xy 133.35 48.26)
+			(xy 123.19 48.26) (xy 133.35 48.26)
 		)
 		(stroke
@@
 	(wire
 		(pts
+			(xy 123.19 49.53) (xy 123.19 48.26)
+		)
+		(stroke
+			(width 0)
+			(type default)
+		)
+	)
+	(wire
+		(pts
 			(xy 27.94 54.61) (xy 25.4 54.61)
 		)
@@
 		(pts
 			(xy 92.71 132.08) (xy 81.28 132.08)
+		)
+		(stroke
+			(width 0)
+			(type default)
+		)
+	)
+	(wire
+		(pts
+			(xy 133.35 58.42) (xy 123.19 58.42)
 		)
 		(stroke
@@
 	)
 	(symbol
+		(lib_id "Device:R")
+		(at 123.19 53.34 0)
+		(unit 1)
+		(body_style 1)
+		(exclude_from_sim no)
+		(in_bom yes)
+		(on_board yes)
+		(in_pos_files yes)
+		(dnp no)
+		(fields_autoplaced yes)
+		(property "Reference" "R15"
+			(at 125.73 52.0699 0)
+			(show_name no)
+			(do_not_autoplace no)
+			(effects
+				(font
+					(size 1.27 1.27)
+				)
+				(justify left)
+			)
+		)
+		(property "Value" "1M"
+			(at 125.73 54.6099 0)
+			(show_name no)
+			(do_not_autoplace no)
+			(effects
+				(font
+					(size 1.27 1.27)
+				)
+				(justify left)
+			)
+		)
+		(property "Footprint" "Resistor_SMD:R_0402_1005Metric"
+			(at 121.412 53.34 90)
+			(hide yes)
+			(show_name no)
+			(do_not_autoplace no)
+			(effects
+				(font
+					(size 1.27 1.27)
+				)
+			)
+		)
+		(property "Datasheet" ""
+			(at 123.19 53.34 0)
+			(hide yes)
+			(show_name no)
+			(do_not_autoplace no)
+			(effects
+				(font
+					(size 1.27 1.27)
+				)
+			)
+		)
+		(property "Description" "Resistor"
+			(at 123.19 53.34 0)
+			(hide yes)
+			(show_name no)
+			(do_not_autoplace no)
+			(effects
+				(font
+					(size 1.27 1.27)
+				)
+			)
+		)
+		(pin "1"
+		)
+		(pin "2"
+		)
+		(instances
+			(project "LEDHeart"
+				(path "/1df9eab6-db71-4fb9-86bd-f1aa227d734a"
+					(reference "R15")
+					(unit 1)
+				)
+			)
+		)
+	)
+	(symbol
 		(lib_id "power:+BATT")
 		(at 19.05 52.07 0)
@@
 	(symbol
 		(lib_id "Device:R")
-		(at 127 48.26 90)
+		(at 119.38 48.26 90)
 		(unit 1)
 		(body_style 1)
@@
 		(fields_autoplaced yes)
 		(property "Reference" "R11"
-			(at 127 41.91 90)
+			(at 119.38 41.91 90)
 			(show_name no)
 			(do_not_autoplace no)
@@
 		)
 		(property "Value" "1K"
-			(at 127 44.45 90)
+			(at 119.38 44.45 90)
 			(show_name no)
 			(do_not_autoplace no)
@@
 		)
 		(property "Footprint" "Resistor_SMD:R_0603_1608Metric_Pad0.98x0.95mm_HandSolder"
-			(at 127 50.038 90)
+			(at 119.38 50.038 90)
 			(hide yes)
 			(show_name no)
@@
 		)
 		(property "Datasheet" ""
-			(at 127 48.26 0)
+			(at 119.38 48.26 0)
 			(hide yes)
 			(show_name no)
@@
 		)
 		(property "Description" "Resistor"
-			(at 127 48.26 0)
-			(hide yes)
-			(show_name no)
+			(at 119.38 48.26 0)
+			(hide yes)
+			(show_name no)
